File: revision0.sch (EAGLE design)
At the start: 95 parts, among them IC1 MSP430FR698X(1)80-PIN_PN, IC3 FT232RL, Q1 32.768 kHz

Commit message: The board is almost done
Connections:
- net ADC-BATT: now also IC1.P9.7/ESICI3/A15/C15; no longer IC1.P4.1/UCB1SOMI/UCB1SCL/ACLK/S4
- net GPS-TIMEPULSE: now also IC1.P9.1/ESICH1/ESITEST1/A9/C9; no longer IC1.P4.0/UCB1SIMO/UCB1SDA/MCLK/S5
- net GPS-WAKEUP: now also IC1.P9.0/ESICH0/ESITEST0/A8/C8; no longer IC1.P4.7/UCB1SOMI/UCB1SCL/TA1.2/S6
- net PWR-USB-SENSE: now also IC1.P4.1/UCB1SOMI/UCB1SCL/ACLK/S4; no longer IC1.P6.3/COM0
- net PWR_GPS_SENSE: now also IC1.P9.6/ESICI2/A14/C14; no longer IC1.P4.6/UCB1SIMO/UCB1SDA/TA1.1/S7
- net SW-CFG-GPS: now also IC1.P9.5/ESICI1/A13/C13, S1.P, S1.P1; no longer IC1.P2.4/TB0.3/COM4/S33, S3.P, S3.P1
- net SW-CHECK-BATT-MEM: now also IC1.P2.0/UCA0SIMO/UCA0TXD/TB0.6/TB0CLK/S14, S3.P, S3.P1; no longer IC1.P2.5/TB0.4/COM5/S32, S1.P, S1.P1
Changed lines of the file:
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@@
 </variantdefs>
 <classes>
-<class number="0" name="default" width="0" drill="0">
+<class number="0" name="signal" width="0.4064" drill="0.4064">
+<clearance class="0" value="0.2034"/>
 </class>
 </classes>
@@
 <net name="GPS-WAKEUP" class="0">
 <segment>
-<wire x1="-7.62" y1="12.7" x2="93.98" y2="12.7" width="0.1524" layer="91"/>
-<label x="96.52" y="12.7" size="1.778" layer="95"/>
-<pinref part="IC1" gate="G$1" pin="P4.7/UCB1SOMI/UCB1SCL/TA1.2/S6"/>
+<wire x1="-7.62" y1="-45.72" x2="-5.08" y2="-48.26" width="0.1524" layer="91"/>
+<wire x1="-5.08" y1="-48.26" x2="93.98" y2="-48.26" width="0.1524" layer="91"/>
+<label x="96.52" y="-45.72" size="1.778" layer="95"/>
+<pinref part="IC1" gate="G$1" pin="P9.0/ESICH0/ESITEST0/A8/C8"/>
 </segment>
 <segment>
@@
 </segment>
 <segment>
-<wire x1="-228.6" y1="2.54" x2="-154.94" y2="2.54" width="0.1524" layer="91"/>
-<pinref part="IC1" gate="G$1" pin="P6.3/COM0"/>
-<label x="-241.3" y="2.54" size="1.778" layer="95"/>
-</segment>
-</net>
-<net name="SW-CHECK-BATT-MEM" class="0">
+<wire x1="-7.62" y1="17.78" x2="93.98" y2="17.78" width="0.1524" layer="91"/>
+<label x="96.52" y="17.78" size="1.778" layer="95"/>
+<pinref part="IC1" gate="G$1" pin="P4.1/UCB1SOMI/UCB1SCL/ACLK/S4"/>
+</segment>
+</net>
+<net name="SW-CFG-GPS" class="0">
 <segment>
 <pinref part="S1" gate="1" pin="P1"/>
@@
 </segment>
 <segment>
-<wire x1="-228.6" y1="-10.16" x2="-154.94" y2="-10.16" width="0.1524" layer="91"/>
-<label x="-241.3" y="-10.16" size="1.778" layer="95"/>
-<pinref part="IC1" gate="G$1" pin="P2.5/TB0.4/COM5/S32"/>
+<label x="96.52" y="-33.02" size="1.778" layer="95"/>
+<pinref part="IC1" gate="G$1" pin="P9.5/ESICI1/A13/C13"/>
+<wire x1="93.98" y1="-33.02" x2="-7.62" y2="-33.02" width="0.1524" layer="91"/>
 </segment>
 </net>
@@
 <net name="PWR_GPS_SENSE" class="0">
 <segment>
-<pinref part="IC1" gate="G$1" pin="P4.6/UCB1SIMO/UCB1SDA/TA1.1/S7"/>
-<wire x1="-7.62" y1="10.16" x2="93.98" y2="10.16" width="0.1524" layer="91"/>
-<label x="96.52" y="10.16" size="1.778" layer="95"/>
+<wire x1="-5.08" y1="-43.18" x2="93.98" y2="-43.18" width="0.1524" layer="91"/>
+<label x="96.52" y="-43.18" size="1.778" layer="95"/>
+<pinref part="IC1" gate="G$1" pin="P9.6/ESICI2/A14/C14"/>
+<wire x1="-5.08" y1="-43.18" x2="-7.62" y2="-30.48" width="0.1524" layer="91"/>
 </segment>
 <segment>
@@
 </segment>
 </net>
-<net name="SW-CFG-GPS" class="0">
+<net name="SW-CHECK-BATT-MEM" class="0">
 <segment>
 <pinref part="S3" gate="1" pin="P1"/>
@@
 </segment>
 <segment>
-<pinref part="IC1" gate="G$1" pin="P2.4/TB0.3/COM4/S33"/>
-<wire x1="-154.94" y1="-7.62" x2="-228.6" y2="-7.62" width="0.1524" layer="91"/>
-<label x="-241.3" y="-7.62" size="1.778" layer="95"/>
+<wire x1="93.98" y1="-73.66" x2="-7.62" y2="-73.66" width="0.1524" layer="91"/>
+<label x="96.52" y="-73.66" size="1.778" layer="95"/>
+<pinref part="IC1" gate="G$1" pin="P2.0/UCA0SIMO/UCA0TXD/TB0.6/TB0CLK/S14"/>
 </segment>
 </net>
@@
 </segment>
 <segment>
-<wire x1="-7.62" y1="15.24" x2="93.98" y2="15.24" width="0.1524" layer="91"/>
-<label x="96.52" y="15.24" size="1.778" layer="95"/>
-<pinref part="IC1" gate="G$1" pin="P4.0/UCB1SIMO/UCB1SDA/MCLK/S5"/>
+<wire x1="-5.08" y1="-45.72" x2="93.98" y2="-45.72" width="0.1524" layer="91"/>
+<label x="96.52" y="-48.26" size="1.778" layer="95"/>
+<pinref part="IC1" gate="G$1" pin="P9.1/ESICH1/ESITEST1/A9/C9"/>
+<wire x1="-5.08" y1="-45.72" x2="-7.62" y2="-43.18" width="0.1524" layer="91"/>
 </segment>
 </net>
@@
 <net name="ADC-BATT" class="0">
 <segment>
-<pinref part="IC1" gate="G$1" pin="P4.1/UCB1SOMI/UCB1SCL/ACLK/S4"/>
-<wire x1="93.98" y1="17.78" x2="-7.62" y2="17.78" width="0.1524" layer="91"/>
-<label x="96.52" y="17.78" size="1.778" layer="95"/>
-</segment>
-<segment>
+<label x="96.52" y="-25.4" size="1.778" layer="95"/>
+<pinref part="IC1" gate="G$1" pin="P9.7/ESICI3/A15/C15"/>
+<wire x1="93.98" y1="-25.4" x2="0" y2="-25.4" width="0.1524" layer="91"/>
+<wire x1="0" y1="-25.4" x2="-7.62" y2="-27.94" width="0.1524" layer="91"/>
+</segment>
+<segment>

Commit message: Added GPS chip, board mostly done, prepare for order
Parts:
- removed C13, C14: 10p, tagps:C-EUC0805
- removed Q1: 32.768 kHz, tagps:XTAL/S
Connections:
- removed net N$4: C14.1, IC1.PJ.4/LFXIN, Q1.2
- removed net N$6: C13.1, IC1.PJ.5/LFXOUT, Q1.1
- net GND: no longer C13.2, C14.2
- net PWR-USB-SENSE: now also IC1.P3.2/UCB1SOMI/UCB1SCL/S27; no longer IC1.P4.1/UCB1SOMI/UCB1SCL/ACLK/S4
- net PWR_GPS_SENSE: now also IC1.P2.3/UCA0STE/TB0OUTH/S17; no longer IC1.P9.6/ESICI2/A14/C14
- net SW-CFG-GPS: now also IC1.P7.0/TA0CLK/S13; no longer IC1.P9.5/ESICI1/A13/C13
Changed lines of the file:
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@@
 </variantdefs>
 <classes>
-<class number="0" name="signal" width="0.4064" drill="0.4064">
+<class number="0" name="signal" width="0.254" drill="0.254">
 <clearance class="0" value="0.2034"/>
 </class>
@@
 <part name="GND11" library="supply1" deviceset="GND" device=""/>
 <part name="P+7" library="tagps" deviceset="VCC" device=""/>
-<part name="Q1" library="tagps" deviceset="XTAL/S" device="" value="32.768 kHz"/>
-<part name="C13" library="tagps" deviceset="C-EU" device="C0805" value="10p"/>
-<part name="C14" library="tagps" deviceset="C-EU" device="C0805" value="10p"/>
-<part name="GND12" library="supply1" deviceset="GND" device=""/>
 <part name="GND13" library="supply1" deviceset="GND" device=""/>
 <part name="R3" library="tagps" deviceset="R-EU_" device="R0805" value="47k"/>
@@
 <instance part="GND11" gate="1" x="30.48" y="-27.94" rot="R90"/>
 <instance part="P+7" gate="VCC" x="30.48" y="-40.64" rot="R270"/>
-<instance part="Q1" gate="G$1" x="68.58" y="-5.08" rot="R270"/>
-<instance part="C13" gate="G$1" x="76.2" y="2.54" rot="MR270"/>
-<instance part="C14" gate="G$1" x="76.2" y="-12.7" rot="MR270"/>
-<instance part="GND12" gate="1" x="93.98" y="-5.08" rot="R90"/>
 <instance part="GND13" gate="1" x="-165.1" y="12.7" rot="R270"/>
 <instance part="R3" gate="G$1" x="-182.88" y="-45.72" rot="R90"/>
@@
 </segment>
 <segment>
-<pinref part="C13" gate="G$1" pin="2"/>
-<wire x1="81.28" y1="2.54" x2="86.36" y2="2.54" width="0.1524" layer="91"/>
-<wire x1="86.36" y1="2.54" x2="86.36" y2="-5.08" width="0.1524" layer="91"/>
-<pinref part="C14" gate="G$1" pin="2"/>
-<wire x1="86.36" y1="-5.08" x2="86.36" y2="-12.7" width="0.1524" layer="91"/>
-<wire x1="86.36" y1="-12.7" x2="81.28" y2="-12.7" width="0.1524" layer="91"/>
-<pinref part="GND12" gate="1" pin="GND"/>
-<wire x1="91.44" y1="-5.08" x2="86.36" y2="-5.08" width="0.1524" layer="91"/>
-<junction x="86.36" y="-5.08"/>
-</segment>
-<segment>
 <pinref part="IC1" gate="G$1" pin="R33/LCDCAP"/>
 <wire x1="-154.94" y1="12.7" x2="-162.56" y2="12.7" width="0.1524" layer="91"/>
@@
 <wire x1="353.06" y1="-66.04" x2="307.34" y2="-66.04" width="0.1524" layer="91"/>
 <label x="353.06" y="-66.04" size="1.778" layer="95"/>
-</segment>
-</net>
-<net name="N$6" class="0">
-<segment>
-<pinref part="IC1" gate="G$1" pin="PJ.5/LFXOUT"/>
-<wire x1="-7.62" y1="0" x2="60.96" y2="0" width="0.1524" layer="91"/>
-<wire x1="60.96" y1="0" x2="60.96" y2="2.54" width="0.1524" layer="91"/>
-<wire x1="60.96" y1="2.54" x2="68.58" y2="2.54" width="0.1524" layer="91"/>
-<pinref part="C13" gate="G$1" pin="1"/>
-<pinref part="Q1" gate="G$1" pin="1"/>
-<wire x1="68.58" y1="2.54" x2="73.66" y2="2.54" width="0.1524" layer="91"/>
-<wire x1="68.58" y1="0" x2="68.58" y2="2.54" width="0.1524" layer="91"/>
-<junction x="68.58" y="2.54"/>
-</segment>
-</net>
-<net name="N$4" class="0">
-<segment>
-<pinref part="IC1" gate="G$1" pin="PJ.4/LFXIN"/>
-<pinref part="C14" gate="G$1" pin="1"/>
-<wire x1="-7.62" y1="-2.54" x2="60.96" y2="-2.54" width="0.1524" layer="91"/>
-<wire x1="60.96" y1="-2.54" x2="60.96" y2="-12.7" width="0.1524" layer="91"/>
-<wire x1="60.96" y1="-12.7" x2="68.58" y2="-12.7" width="0.1524" layer="91"/>
-<pinref part="Q1" gate="G$1" pin="2"/>
-<wire x1="68.58" y1="-12.7" x2="73.66" y2="-12.7" width="0.1524" layer="91"/>
-<wire x1="68.58" y1="-10.16" x2="68.58" y2="-12.7" width="0.1524" layer="91"/>
-<junction x="68.58" y="-12.7"/>
 </segment>
 </net>
@@
 </segment>
 <segment>
-<wire x1="-7.62" y1="17.78" x2="93.98" y2="17.78" width="0.1524" layer="91"/>
-<label x="96.52" y="17.78" size="1.778" layer="95"/>
-<pinref part="IC1" gate="G$1" pin="P4.1/UCB1SOMI/UCB1SCL/ACLK/S4"/>
+<wire x1="-162.56" y1="-22.86" x2="-154.94" y2="-22.86" width="0.1524" layer="91"/>
+<pinref part="IC1" gate="G$1" pin="P3.2/UCB1SOMI/UCB1SCL/S27"/>
+<wire x1="-162.56" y1="-22.86" x2="-162.56" y2="-10.16" width="0.1524" layer="91"/>
+<wire x1="-162.56" y1="-10.16" x2="-228.6" y2="-10.16" width="0.1524" layer="91"/>
+<label x="-241.3" y="-10.16" size="1.778" layer="95"/>
 </segment>
 </net>
@@
 </segment>
 <segment>
-<label x="96.52" y="-33.02" size="1.778" layer="95"/>
-<pinref part="IC1" gate="G$1" pin="P9.5/ESICI1/A13/C13"/>
-<wire x1="93.98" y1="-33.02" x2="-7.62" y2="-33.02" width="0.1524" layer="91"/>
+<label x="96.52" y="-76.2" size="1.778" layer="95"/>
+<wire x1="93.98" y1="-76.2" x2="-2.54" y2="-76.2" width="0.1524" layer="91"/>
+<pinref part="IC1" gate="G$1" pin="P7.0/TA0CLK/S13"/>
+<wire x1="-2.54" y1="-76.2" x2="-7.62" y2="-71.12" width="0.1524" layer="91"/>
 </segment>
 </net>
@@
 <net name="PWR_GPS_SENSE" class="0">
 <segment>
-<wire x1="-5.08" y1="-43.18" x2="93.98" y2="-43.18" width="0.1524" layer="91"/>
+<wire x1="-233.68" y1="-71.12" x2="-160.02" y2="-71.12" width="0.1524" layer="91"/>
 <label x="96.52" y="-43.18" size="1.778" layer="95"/>
-<pinref part="IC1" gate="G$1" pin="P9.6/ESICI2/A14/C14"/>
-<wire x1="-5.08" y1="-43.18" x2="-7.62" y2="-30.48" width="0.1524" layer="91"/>
+<wire x1="-160.02" y1="-71.12" x2="-160.02" y2="-68.58" width="0.1524" layer="91"/>
+<pinref part="IC1" gate="G$1" pin="P2.3/UCA0STE/TB0OUTH/S17"/>
+<wire x1="-160.02" y1="-68.58" x2="-154.94" y2="-68.58" width="0.1524" layer="91"/>
+<label x="-238.76" y="-71.12" size="1.778" layer="95"/>
 </segment>
 <segment>
@@
 </segment>
 <segment>
-<wire x1="93.98" y1="-73.66" x2="-7.62" y2="-73.66" width="0.1524" layer="91"/>
-<label x="96.52" y="-73.66" size="1.778" layer="95"/>
+<wire x1="93.98" y1="-78.74" x2="-2.54" y2="-78.74" width="0.1524" layer="91"/>
+<wire x1="-2.54" y1="-78.74" x2="-7.62" y2="-73.66" width="0.1524" layer="91"/>
+<label x="96.52" y="-78.74" size="1.778" layer="95"/>
 <pinref part="IC1" gate="G$1" pin="P2.0/UCA0SIMO/UCA0TXD/TB0.6/TB0CLK/S14"/>
 </segment>
